File: Schematic and PCB/USB_to_UART.kicad_sch (KiCad schematic)
At the start: 19 parts, among them J1 USB_B_Micro, Q1 NPN, Q2 NPN, U2 FT232RL

Commit message: Schematic update uart and power supply
Parts:
- removed R3, R4: 27R, symbol Device:R
Connections:
- net D+: now also C2.1, D3.2 (A2), J1.3 (D+)
- net D-: now also C3.1, D4.2 (A2), J1.2 (D-)
- net DTR: now also U2.2 (DTR)
- net GND: now also U2.26 (TEST)
- net RTS: now also U2.3 (RTS)
- net TXD: now reaches U2.1 (TXD)
- net RXD: now reaches U2.5 (RXD)
- no-connect marks 3 -> 4
Changed lines of the file:
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@@
 		(at 139.7 118.11)
 	)
+	(no_connect
+		(at 139.7 113.03)
+	)
 	(wire
 		(pts
@@
 	(wire
 		(pts
+			(xy 138.43 130.81) (xy 138.43 142.24)
+		)
+		(stroke
+			(width 0)
+			(type default)
+		)
+	)
+	(wire
+		(pts
 			(xy 43.18 147.32) (xy 43.18 162.56)
 		)
@@
 	(wire
 		(pts
+			(xy 180.34 105.41) (xy 181.61 105.41)
+		)
+		(stroke
+			(width 0)
+			(type default)
+		)
+	)
+	(wire
+		(pts
 			(xy 154.94 138.43) (xy 154.94 140.97)
 		)
@@
 	(wire
 		(pts
-			(xy 81.28 34.29) (xy 96.52 34.29)
+			(xy 81.28 34.29) (xy 97.79 34.29)
 		)
 		(stroke
@@
 	(wire
 		(pts
-			(xy 104.14 36.83) (xy 105.41 36.83)
-		)
-		(stroke
-			(width 0)
-			(type default)
-		)
-	)
-	(wire
-		(pts
 			(xy 36.83 36.83) (xy 69.85 36.83)
 		)
@@
 	(wire
 		(pts
-			(xy 93.98 36.83) (xy 96.52 36.83)
+			(xy 93.98 36.83) (xy 97.79 36.83)
 		)
 		(stroke
@@
 	(wire
 		(pts
+			(xy 139.7 130.81) (xy 138.43 130.81)
+		)
+		(stroke
+			(width 0)
+			(type default)
+		)
+	)
+	(wire
+		(pts
+			(xy 180.34 95.25) (xy 181.61 95.25)
+		)
+		(stroke
+			(width 0)
+			(type default)
+		)
+	)
+	(wire
+		(pts
+			(xy 180.34 97.79) (xy 187.96 97.79)
+		)
+		(stroke
+			(width 0)
+			(type default)
+		)
+	)
+	(wire
+		(pts
 			(xy 36.83 29.21) (xy 40.64 29.21)
 		)
@@
 	(wire
 		(pts
-			(xy 104.14 34.29) (xy 105.41 34.29)
-		)
-		(stroke
-			(width 0)
-			(type default)
-		)
-	)
-	(wire
-		(pts
 			(xy 81.28 52.07) (xy 81.28 55.88)
 		)
@@
 		(pts
 			(xy 72.39 168.91) (xy 64.77 168.91)
+		)
+		(stroke
+			(width 0)
+			(type default)
+		)
+	)
+	(wire
+		(pts
+			(xy 180.34 100.33) (xy 181.61 100.33)
 		)
 		(stroke
@@
 		)
 	)
+	(global_label "TXD"
+		(shape output)
+		(at 181.61 95.25 0)
+		(fields_autoplaced yes)
+		(effects
+			(font
+				(size 1.27 1.27)
+			)
+			(justify left)
+		)
+		(property "Intersheetrefs" "${INTERSHEET_REFS}"
+			(at 188.0423 95.25 0)
+			(effects
+				(font
+					(size 1.27 1.27)
+				)
+				(justify left)
+				(hide yes)
+			)
+		)
+	)
 	(global_label "D+"
 		(shape bidirectional)
@@
 	(global_label "D+"
 		(shape bidirectional)
-		(at 105.41 34.29 0)
+		(at 97.79 34.29 0)
 		(fields_autoplaced yes)
 		(effects
@@
 		)
 		(property "Intersheetrefs" "${INTERSHEET_REFS}"
-			(at 112.3489 34.29 0)
+			(at 104.7289 34.29 0)
 			(effects
 				(font
@@
 		)
 	)
+	(global_label "DTR"
+		(shape output)
+		(at 181.61 105.41 0)
+		(fields_autoplaced yes)
+		(effects
+			(font
+				(size 1.27 1.27)
+			)
+			(justify left)
+		)
+		(property "Intersheetrefs" "${INTERSHEET_REFS}"
+			(at 188.1028 105.41 0)
+			(effects
+				(font
+					(size 1.27 1.27)
+				)
+				(justify left)
+				(hide yes)
+			)
+		)
+	)
 	(global_label "3V3OUT"
 		(shape input)
@@
 		)
 	)
+	(global_label "RXD"
+		(shape input)
+		(at 187.96 97.79 0)
+		(fields_autoplaced yes)
+		(effects
+			(font
+				(size 1.27 1.27)
+			)
+			(justify left)
+		)
+		(property "Intersheetrefs" "${INTERSHEET_REFS}"
+			(at 194.6947 97.79 0)
+			(effects
+				(font
+					(size 1.27 1.27)
+				)
+				(justify left)
+				(hide yes)
+			)
+		)
+	)
 	(global_label "RTS"
 		(shape input)
@@
 	(global_label "D-"
 		(shape bidirectional)
-		(at 105.41 36.83 0)
+		(at 97.79 36.83 0)
 		(fields_autoplaced yes)
 		(effects
@@
 		)
 		(property "Intersheetrefs" "${INTERSHEET_REFS}"
-			(at 112.3489 36.83 0)
+			(at 104.7289 36.83 0)
 			(effects
 				(font
@@
 				)
 				(justify left)
-				(hide yes)
-			)
-		)
-	)
-	(global_label "3V3OUT"
-		(shape input)
-		(at 127 111.76 180)
-		(fields_autoplaced yes)
-		(effects
-			(font
-				(size 1.27 1.27)
-			)
-			(justify right)
-		)
-		(property "Intersheetrefs" "${INTERSHEET_REFS}"
-			(at 116.8786 111.76 0)
-			(effects
-				(font
-					(size 1.27 1.27)
-				)
-				(justify right)
 				(hide yes)
 			)
@@
 				(path "/97687706-6280-4d24-828f-729b51ecbb36/10b1fa72-c369-45a6-b778-9504a607a8f3"
 					(reference "#PWR08")
-					(unit 1)
-				)
-			)
-		)
-	)
-	(symbol
-		(lib_id "Device:R")
-		(at 100.33 36.83 270)
-		(mirror x)
-		(unit 1)
-		(exclude_from_sim no)
-		(in_bom yes)
-		(on_board yes)
-		(dnp no)
-		(property "Reference" "R4"
-			(at 100.33 43.18 90)
-			(effects
-				(font
-					(size 1.27 1.27)
-				)
-			)
-		)
-		(property "Value" "27R"
-			(at 100.33 40.64 90)
-			(effects
-				(font
-					(size 1.27 1.27)
-				)
-			)
-		)
-		(property "Footprint" ""
-			(at 100.33 38.608 90)
-			(effects
-				(font
-					(size 1.27 1.27)
-				)
-				(hide yes)
-			)
-		)
-		(property "Datasheet" "~"
-			(at 100.33 36.83 0)
-			(effects
-				(font
-					(size 1.27 1.27)
-				)
-				(hide yes)
-			)
-		)
-		(property "Description" "Resistor"
-			(at 100.33 36.83 0)
-			(effects
-				(font
-					(size 1.27 1.27)
-				)
-				(hide yes)
-			)
-		)
-		(pin "1"
-		)
-		(pin "2"
-		)
-		(instances
-			(project "RC_Car_PWR"
-				(path "/97687706-6280-4d24-828f-729b51ecbb36/10b1fa72-c369-45a6-b778-9504a607a8f3"
-					(reference "R4")
 					(unit 1)
 				)
@@
 	)
 	(symbol
-		(lib_id "Device:R")
-		(at 100.33 34.29 90)
-		(unit 1)
-		(exclude_from_sim no)
-		(in_bom yes)
-		(on_board yes)
-		(dnp no)
-		(fields_autoplaced yes)
-		(property "Reference" "R3"
-			(at 100.33 27.94 90)
-			(effects
-				(font
-					(size 1.27 1.27)
-				)
-			)
-		)
-		(property "Value" "27R"
-			(at 100.33 30.48 90)
-			(effects
-				(font
-					(size 1.27 1.27)
-				)
-			)
-		)
-		(property "Footprint" ""
-			(at 100.33 36.068 90)
-			(effects
-				(font
-					(size 1.27 1.27)
-				)
-				(hide yes)
-			)
-		)
-		(property "Datasheet" "~"
-			(at 100.33 34.29 0)
-			(effects
-				(font
-					(size 1.27 1.27)
-				)
-				(hide yes)
-			)
-		)
-		(property "Description" "Resistor"
-			(at 100.33 34.29 0)
-			(effects
-				(font
-					(size 1.27 1.27)
-				)
-				(hide yes)
-			)
-		)
-		(pin "1"
-		)
-		(pin "2"
-		)
-		(instances
-			(project "RC_Car_PWR"
-				(path "/97687706-6280-4d24-828f-729b51ecbb36/10b1fa72-c369-45a6-b778-9504a607a8f3"
-					(reference "R3")
-					(unit 1)
-				)
-			)
-		)
-	)
-	(symbol
 		(lib_id "power:GND")
 		(at 52.07 57.15 0)
@@
 					(unit 1)
 				)
+			)
+		)
+	)
+	(symbol
+		(lib_id "power:GND")
+		(at 138.43 142.24 0)
+		(unit 1)
+		(exclude_from_sim no)
+		(in_bom yes)
+		(on_board yes)
+		(dnp no)
+		(fields_autoplaced yes)
+		(property "Reference" "#PWR010"
+			(at 138.43 148.59 0)
+			(effects
+				(font
+					(size 1.27 1.27)
+				)
+				(hide yes)
+			)
+		)
+		(property "Value" "GND"
+			(at 138.43 147.32 0)
+			(effects
+				(font
+					(size 1.27 1.27)
+				)
+			)
+		)
+		(property "Footprint" ""
+			(at 138.43 142.24 0)
+			(effects
+				(font
+					(size 1.27 1.27)
+				)
+				(hide yes)
+			)
+		)
+		(property "Datasheet" ""
+			(at 138.43 142.24 0)
+			(effects
+				(font
+					(size 1.27 1.27)
+				)
+				(hide yes)
+			)
+		)
+		(property "Description" "Power symbol creates a global label with name \"GND\" , ground"
+			(at 138.43 142.24 0)
+			(effects
+				(font
+					(size 1.27 1.27)
+				)
+				(hide yes)
+			)
+		)
+		(pin "1"
+		)
+		(instances
+			(project "RC_Car_PWR"
+				(path "/97687706-6280-4d24-828f-729b51ecbb36/10b1fa72-c369-45a6-b778-9504a607a8f3"
+					(reference "#PWR010")
+					(unit 1)
+				)

Commit message: diff pair
Other:
- note added: "diff pair"
Changed lines of the file:
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@@
+		)
+	)
+	(rectangle
+		(start 95.25 31.75)
+		(end 106.68 39.37)
+		(stroke
+			(width 0)
+			(type dash)
+			(color 255 0 0 1)
+		)
+		(fill
+			(type none)
+		)
+	)
+	(text "diff pair"
+		(exclude_from_sim no)
+		(at 101.092 30.48 0)
+		(effects
+			(font
+				(size 1.27 1.27)
+				(color 255 0 0 1)
+			)
 		)
 	)
